File: pcb/amatelus73.kicad_pcb (KiCad board)
At the start: 2 copper layers, 361.9 x 104.8 mm, 237 parts, among them J1 Conn_01x04, J2 AudioJack4, SW1 SW_PUSH, SW10 SW_PUSH, SW11 SW_PUSH, SW12 SW_PUSH, SW13 SW_PUSH, SW14 SW_PUSH, SW15 SW_PUSH, SW16 SW_PUSH, SW17 SW_PUSH, SW18 SW_PUSH, SW19 SW_PUSH, SW2 SW_PUSH, SW20 SW_PUSH, SW21 SW_PUSH, SW22 SW_PUSH, SW23 SW_PUSH, SW24 SW_PUSH, SW25 SW_PUSH, SW26 SW_PUSH, SW27 SW_PUSH, SW28 SW_PUSH, SW29 SW_PUSH, SW3 SW_PUSH, SW30 SW_PUSH, SW31 SW_PUSH, SW32 SW_PUSH, SW33 SW_PUSH, SW34 SW_PUSH, SW35 SW_PUSH, SW36 SW_PUSH, SW37 SW_PUSH, SW38 SW_PUSH, SW39 SW_PUSH, SW4 SW_PUSH, SW40 SW_PUSH, SW41 SW_PUSH, SW42 SW_PUSH, SW43 SW_PUSH, SW44 SW_PUSH, SW45 SW_PUSH, SW46 SW_PUSH, SW47 SW_PUSH, SW48 SW_PUSH, SW49 SW_PUSH, SW5 SW_PUSH, SW50 SW_PUSH, SW51 SW_PUSH, SW52 SW_PUSH, SW53 SW_PUSH, SW54 SW_PUSH, SW55 SW_PUSH, SW56 SW_PUSH, SW57 SW_PUSH, SW58 SW_PUSH, SW59 SW_PUSH, SW6 SW_PUSH, SW60 SW_PUSH, SW61 SW_PUSH, SW62 SW_PUSH, SW63 SW_PUSH, SW64 SW_PUSH, SW65 SW_PUSH, SW66 SW_PUSH, SW67 SW_PUSH, SW68 SW_PUSH, SW69 SW_PUSH, SW7 SW_PUSH, SW70 SW_PUSH, SW71 SW_PUSH, SW72 SW_PUSH, SW73 SW_PUSH, SW74 SW_PUSH, SW8 SW_PUSH, SW9 SW_PUSH, U1 ProMicro_r

Commit message: 2nd order
Parts:
- SW74: footprint keyboard:tact_switch2 -> Button_Switch_THT:SW_Tactile_SPST_Angled_PTS645Vx31-2LFS
- moved SW74 2.56 mm to (378.5, 41.9)
- moved J1 2.22 mm to (361.3, 61.0)
- moved L40 2.22 mm to (185.7, 73.7)
- moved D16 2.04 mm to (322.6, 41.9), turned to 180 degrees
Routing:
- net VCC: track 1746.9 -> 1756.5 mm
- net GND: track 1796.4 -> 1799.2 mm
- net Net-(L40-Pad2): track 12.1 -> 14.4 mm
- net SCL: track 71.5 -> 73.7 mm
- net RST: track 27.1 -> 26.1 mm
- net ROW1: track 357.7 -> 358.6 mm
- net Net-(L39-Pad2): track 11.4 -> 12.3 mm
- net ROW4: track 384.9 -> 385.8 mm
- net COL6: track 266.0 -> 266.7 mm
- net Net-(D16-Pad1): track 3.71 -> 4.25 mm

Commit message: fix silk
Parts:
- L1, L10, L11, L12, L13, L14, L15, L16, L17, L18, L19, L2, L20, L21, L22, L23, L24, L25, L26, L27, L28, L29, L3, L30, L31, L32, L33, L34, L35, L36, L37, L38, L39, L4, L40, L41, L42, L43, L44, L45, L46, L47, L48, L49, L5, L50, L51, L52, L53, L54, L55, L56, L57, L58, L59, L6, L60, L61, L62, L63, L64, L65, L66, L67, L68, L69, L7, L70, L71, L72, L73, L74, L8, L9: footprint keyboard:YS-SK6812MINI-E -> Keyboard:YS-SK6812MINI-E
- SW1, SW10, SW11, SW12, SW13, SW14, SW15, SW17, SW19, SW2, SW20, SW21, SW22, SW23, SW24, SW25, SW26, SW27, SW28, SW29, SW3, SW30, SW32, SW34, SW35, SW36, SW37, SW38, SW39, SW4, SW40, SW41, SW42, SW43, SW44, SW45, SW48, SW49, SW5, SW50, SW51, SW52, SW53, SW54, SW55, SW56, SW57, SW58, SW59, SW6, SW60, SW61, SW63, SW7, SW71, SW72, SW73, SW8, SW9: footprint keyboard:MX_Hotswap_1u -> Keyboard:MX_Hotswap_1u
- SW16: footprint keyboard:MX_Hotswap_2u_Reversed -> Keyboard:MX_Hotswap_2u_Reversed
- SW18, SW31: footprint keyboard:MX_Hotswap_1.5u -> Keyboard:MX_Hotswap_1.5u
- SW33: footprint keyboard:MX_Hotswap_1.75u -> Keyboard:MX_Hotswap_1.75u
- SW46, SW47: footprint keyboard:MX_Hotswap_2.25u -> Keyboard:MX_Hotswap_2.25u
- SW62: footprint keyboard:MX_Hotswap_2.75u -> Keyboard:MX_Hotswap_2.75u
- SW64, SW65, SW66, SW67, SW68, SW69, SW70: footprint keyboard:MX_Hotswap_1.25u -> Keyboard:MX_Hotswap_1.25u
